File: doc/hardware/kicad/schemas/arlyPhone/arlyPhone.kicad_sch (KiCad schematic)
At the start: 0 parts

Commit message: alimentations + preamplier
Parts:
- added C1, C2, C3: 470n, symbol Device:C
- added C10, C4, C8: 100n, symbol Device:C
- added C11, C5, C7, C9: 10u, symbol Device:C
- added C6: 22u, symbol Device:C_Small_US
- added D1: 1N4148W, Diode_SMD:D_SOD-123, symbol Diode:1N4148W
- added D2, D3: LED, symbol Device:LED
- added J1: Conn_01x02_Pin, symbol Connector:Conn_01x02_Pin
- added MK1: Microphone, symbol Device:Microphone
- added P1: USB_C_Plug_USB2.0, symbol Connector:USB_C_Plug_USB2.0
- added R1, R6, R7: 1k, symbol Device:R_US
- added R2: 47k, symbol Device:R_US
- added R3, R4: 10k, symbol Device:R_US
- added R5: 1M, symbol Device:R_US
- added R8: 1k2, symbol Device:R_US
- added SW1, SW2: bp, symbol Switch:SW_Push_Dual_x2
- added U1: NJM5532, symbol Amplifier_Operational:NJM5532
- added U2: TP4056-42-ESOP8, Package_SO:SOIC-8-1EP_3.9x4.9mm_P1.27mm_EP2.41x3.3mm_ThermalVias, symbol Battery_Management:TP4056-42-ESOP8
- added U3: AMS1117-3.3, Package_TO_SOT_SMD:SOT-223-3_TabPin2, symbol Regulator_Linear:AMS1117-3.3
- added U4: PAM8403D, Package_SO:SOIC-16_3.9x9.9mm_P1.27mm, symbol Amplifier_Audio:PAM8403D
Connections:
- new net: C1.1, C2.1, MK1.2 (+), R1.2
- new net: C1.2, C2.2, R2.1
- new net: R8.1, U2.2 (PROG)
- new net: C7.2, D1.1 (K), D2.2 (A), D3.2 (A), U2.4 (V_{CC}), U2.8 (CE)
- new net: R6.2, U2.6 (~{STDBY})
- new net: R7.2, U2.7 (~{CHRG})
- new net: C3.1, R2.2, R5.1, U1.2 (-)
- new net: D3.1 (K), R7.1
- new net: SW1.1 (C), SW1.3 (C)
- new net: SW1.2 (D), SW1.4 (D)
- new net: R3.2, R4.1, U1.3 (+)
- new net: D2.1 (K), R6.1
- new net: D1.2 (A), P1.A4 (VBUS), P1.A9 (VBUS), P1.B4 (VBUS), P1.B9 (VBUS)
- new net: U4.13 (PVDD), U4.4 (PVDD)
- new net: U4.15 (PGND), U4.2 (PGND)
- new net +3.3V: C10.1, C11.1, U3.2 (VO)
- new net +5V: C4.2, C5.2, C6.1, C8.1, C9.1, J1.2 (Pin_2), R1.1, R3.1, U1.8 (V+), U2.5 (BAT), U3.3 (VI)
- new net GND: C10.2, C11.2, C4.1, C5.1, C6.2, C7.1, C8.2, C9.2, J1.1 (Pin_1), MK1.1 (-), P1.A1 (GND), P1.A12 (GND), P1.B1 (GND), P1.B12 (GND), P1.SH (SHIELD), R4.2, R8.2, U1.4 (V-), U2.1 (TEMP), U2.3 (GND), U3.1 (GND)
- new net Micro_ADC: C3.2, R5.2, U1.1
Other:
- company: (none) -> Integre trvailleure
- title: (none) -> arlyPhone

Commit message: mcu
Parts:
- removed SW1, SW2: bp, symbol Switch:SW_Push_Dual_x2

Commit message: suite
Parts:
- removed J1: Conn_01x02_Pin, symbol Connector:Conn_01x02_Pin
- added C12, C13, C14, C21, C22, C23: 470n, symbol Device:C
- added C15, C19: 10u, symbol Device:C
- added C16, C17, C18: 1u, symbol Device:C
- added C20: 22u, symbol Device:C_Small_US
- added C24, C25, C26: 22u, symbol Device:C
- added J1, J2: Conn_01x01_Pin, symbol Connector:Conn_01x01_Pin
- added J? (x2): Conn_01x02_Pin, symbol Connector:Conn_01x02_Pin
- added R10, R9: 20k, symbol Device:R_US
- added R11, R13, R14, R16: 10k, symbol Device:R_US
- added R12: 47k, symbol Device:R_US
- added R15: 1M, symbol Device:R_US
- added SW1, SW10, SW11, SW12, SW13, SW14, SW15, SW16, SW17, SW18, SW19, SW2, SW20, SW21, SW22, SW23, SW24, SW3, SW4, SW5, SW6, SW7, SW8, SW9: SW_Push, symbol Switch:SW_Push
- added U5: STM32F103C8Tx, Package_QFP:LQFP-48_7x7mm_P0.5mm, symbol MCU_ST_STM32F1:STM32F103C8Tx
Connections:
- net +3.3V: now also U5.1 (VBAT), U5.24 (VDD), U5.36 (VDD), U5.48 (VDD), U5.9 (VDDA)
- net +5V: now also U4.12 (~{SHDN}), U4.13 (PVDD), U4.4 (PVDD), U4.5 (~{MUTE}), U4.6 (VDD), C15.1, C16.1, C17.1, C18.1, C19.1, C20.1, C24.1, C25.1, C26.1, J1.1 (Pin_1), R11.1, R13.1
- net GND: now also U4.11 (GND), U4.15 (PGND), U4.2 (PGND), C13.2, C15.2, C16.2, C17.2, C18.2, C19.2, C20.2, C24.2, C25.2, C26.2, J2.1 (Pin_1), R14.2, R16.1, U5.23 (VSS), U5.35 (VSS), U5.47 (VSS), U5.8 (VSSA)
- net at U1.5 (+): now also R13.2, R14.1
- net at U1.6 (-): now also C23.1, R12.2, R15.1
- net jack: now reaches U1.7
- net jack: now also C23.2, R15.2
- net at U4.1 (LOUT+): now also J?.2 (Pin_2)
- net at U4.10 (INR): now also R10.2
- net at U4.14 (ROUT-): now also J?.2 (Pin_2)
- net at U4.16 (ROUT+): now also J?.1 (Pin_1)
- net at U4.3 (LOUT-): now also J?.1 (Pin_1)
- net at U4.7 (INL): now also R9.2
- net at U4.8 (VREF): now also C13.1
- new net: C12.2, R9.1
- new net: C21.2, C22.2, R12.1
- new net: C14.2, R10.1
- new net: R16.2, U5.20 (PB2)
- new net Col1: SW1.2, SW13.2, SW17.2, SW21.2, SW5.2, SW9.2
- new net Col2: SW10.2, SW14.2, SW18.2, SW2.2, SW22.2, SW6.2
- new net Col3: SW11.2, SW15.2, SW19.2, SW23.2, SW3.2, SW7.2
- new net Col4: SW12.2, SW16.2, SW20.2, SW24.2, SW4.2, SW8.2
- new net HP_PWM: C12.1, C14.1, C21.1, C22.1, R11.2
- new net Ligne_1: SW1.1, SW2.1, SW3.1, SW4.1
- new net Ligne_2: SW5.1, SW6.1, SW7.1, SW8.1
- new net Ligne_3: SW10.1, SW11.1, SW12.1, SW9.1
- new net Ligne_4: SW13.1, SW14.1, SW15.1, SW16.1
- new net Ligne_5: SW17.1, SW18.1, SW19.1, SW20.1
- new net Ligne_6: SW21.1, SW22.1, SW23.1, SW24.1
- no-connect marks 0 -> 1
Other:
- moved on the sheet: U4

Commit message: SCHEMA GENERAL
Parts:
- added C27, C28: 22p, symbol Device:C
- added C29, C30: 8p, symbol Device:C
- added R17: 100K, symbol Device:R_US
- added SW25, SW26: SW_Push, symbol Switch:SW_Push
- added Y1: 8Mhz, symbol Device:Crystal
- added Y2: 32.768Khz, symbol Device:Crystal
Connections:
- net GND: now also C27.1, C28.1, C29.1, C30.1
- new net: R17.1, SW25.2
- new net PC14: C29.2, Y2.2
- new net PC15: C30.2, Y2.1
- new net PD0: C27.2, Y1.2
- new net PD1: C28.2, Y1.1
